Commit message: Uploaded a controller and utils
- Added the kinematics controller of the robot based on real parameters
- Added a waypoint tracking using the kinematics controller

File: mscbot_description/urdf/mscbot.urdf.xacro (robot description, xacro)
@@ -1,14 +1,21 @@
 <?xml version="1.0"?>
 <robot xmlns:xacro="http://www.ros.org/wiki/xacro" name="robot_name">
-    <xacro:include filename="mscbot.xacro"/>
-    <xacro:include filename="mscbot_gazebo.xacro"/>
-    <xacro:include filename="mscbot_ros2_control.xacro"/>
+     <!-- insert the gazebo properties and control -->
+     <xacro:include filename="mscbot.xacro"/>
+     <xacro:include filename="mscbot_gazebo.xacro"/>
+     <xacro:include filename="mscbot_ros2_control.xacro"/>
     <!-- Base link -->
     <link name="base_link" />
-    <link name="orientation_link" />
+    <link name="orientation_link" >
+        <inertial>
+            <mass value="100.0"/>
+            <origin xyz="0 0 0"/>
+            <inertia ixx="0.0001" ixy="0.0" ixz="0.0" iyy="0.0001" iyz="0.0" izz="0.0001"/>
+          </inertial>
+    </link>
     <joint name="orientation_joint" type="fixed">
         <parent link="base_link"/>
         <child link="orientation_link"/>
-        <origin xyz="0 0 0" rpy="0 0 0"/>
+        <origin xyz="0 0 105.0e-3" rpy="0 0 0"/>
     </joint>
     <!-- inserting motors and wheels -->

File: mscbot_description/urdf/mscbot.xacro (robot description, xacro)
@@ -137,5 +137,5 @@
             <parent link="caster_wheel_base"/>
             <child link="caster_wheel_top_plate_link"/>
-            <origin xyz="-143.158e-3 0 0" rpy="0 0 0"/>
+            <origin xyz="-143.158e-3 0 1.0e-3" rpy="0 0 0"/>
         </joint>
         <!-- Upper part -->
@@ -157,8 +157,9 @@
             </inertial>
         </link>
-        <joint name="chassis_to_caster_wheel_upper_part_joint" type="fixed">
+        <joint name="chassis_to_caster_wheel_upper_part_joint" type="continuous">
             <parent link="caster_wheel_top_plate_link"/>
             <child link="caster_wheel_upper_part_link"/>
             <origin xyz="-10.0e-3 0 -17.13636e-3" rpy="0 0 0"/>
+            <axis xyz="0 0 1" />
         </joint>
         <!-- Caster Wheel -->

File: mscbot_description/urdf/mscbot_gazebo.xacro (robot description, xacro)
@@ -34,18 +34,20 @@
     </gazebo>
     <gazebo reference="caster_wheel_upper_part_link">
-        <mu1>0.1</mu1>
-        <mu2>0.1</mu2>
+        <mu1>1.0</mu1>
+        <mu2>1.0</mu2>
         <kp>100000000.0</kp>
         <kd>100.0</kd>
         <minDepth>0.001</minDepth>
         <maxVel>0.1</maxVel>
+        <fdir1>0 0 1</fdir1>
     </gazebo>
     <gazebo reference="caster_wheel_link">
-        <mu1>0.1</mu1>
-        <mu2>0.1</mu2>
-        <kp>100000000.0</kp>
-        <kd>100.0</kd>
+        <mu1>100000000000000.0</mu1>
+        <mu2>100000000000000.0</mu2>
+        <kp>10000000000000.0</kp>
+        <kd>10.0</kd>
         <minDepth>0.001</minDepth>
         <maxVel>0.1</maxVel>
+        <fdir1>0 1 0</fdir1>
     </gazebo>
     <!-- ROS 2 Control -->
