Commit message: Added wheel slip plugin and uploaded the wp tracking

File: mscbot_description/urdf/components/mscbot_gazebo.xacro (robot description, xacro)
@@ -59,3 +59,17 @@
       </plugin>
     </gazebo>
+    <plugin name="wheel_slip_controller" filename="libgazebo_ros_wheel_slip.so">
+        <mu1>1.0</mu1>
+        <mu2>0.8</mu2>
+        <slip_compliance_unitless_lateral>0.0</slip_compliance_unitless_lateral>
+        <slip_compliance_unitless_longitudinal>0.0</slip_compliance_unitless_longitudinal>
+        <wheel_link_name>left_wheel_link</wheel_link_name>
+    </plugin>
+    <plugin name="wheel_slip_controller" filename="libgazebo_ros_wheel_slip.so">
+        <mu1>1.0</mu1>
+        <mu2>0.8</mu2>
+        <slip_compliance_unitless_lateral>0.0</slip_compliance_unitless_lateral>
+        <slip_compliance_unitless_longitudinal>0.0</slip_compliance_unitless_longitudinal>
+        <wheel_link_name>right_wheel_link</wheel_link_name>
+    </plugin>
 </robot>

File: mscbot_description/urdf/mscbot.urdf.xacro (robot description, xacro)
@@ -10,5 +10,5 @@
     <link name="orientation_link" >
         <inertial>
-            <mass value="100.0"/>
+            <mass value="400.0"/>
             <origin xyz="0 0 0"/>
             <inertia ixx="0.0001" ixy="0.0" ixz="0.0" iyy="0.0001" iyz="0.0" izz="0.0001"/>
